File: adafruit_tricket_m0/Trinket M0 template.brd (EAGLE design)
At the start: 160 x 100 mm, 1 part

Commit message: big push
Parts:
- removed LED1: (no value), adafruit:SEGMENT_BL-M15A881
- added JP3, JP4: (no value), microbuilder:1X05_ROUND_76
Other:
- board outline removed
- board text added: "D0/A4/SDA"
- board text added: "D1/A0/VOUT"
- board text added: "D2/A1/SCL/MISO"
- board text added: "D3/A3/TXD/SCK"
- board text added: "D4/A2/RXD/MOSI"
